File: Circuits/Boards R3/Swarm Board_3.sch (EAGLE design)
At the start: 139 parts, among them CON1 ISP(2X3), CON2 MAIN_CONNECTOR_14SMD, CON4 HEADER_3X1, CON5 HEADER_3X1, CON7 MAIN_CONNECTOR_8, M1 VIBMOTOR, T1 TEFT4300, T10 TEFT4300, T11 NPN2N2222, T12 SI2333DS-T1, T13 NPN2N2222, T14 NPN2N2222, T15 NPN2N2222, T16 NPN2N2222, T17 NPN2N2222, T18 NPN2N2222, T19 IRLML6244TR, T2 TEFT4300, T20 IRLML6244TR, T21 IRLML6244TR, T22 IRLML6244TR, T23 IRLML6244TR, T3 NPN2N2222, T4 TEFT4300, T5 TEFT4300, T6 TEFT4300, T7 TEFT4300, T8 TEFT4300, T9 TEFT4300, U1 ATMEGA324P, U2 MCP73833, U3 ATMEGA1281, U4 MCP9700A, U5 AH182, U6 AH182, U7 QRE1113, U8 QRE1113, U9 QRE1113

Commit message: more
Parts:
- removed R25, R6: 50k, Passive:RES0603
Connections:
- net +VSENSE: no longer R25.2, R6.2
- net ENCA: no longer R25.1
- net ENCB: no longer R6.1
Changed lines of the file:
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@@
 <?xml version="1.0" encoding="utf-8"?>
 <!DOCTYPE eagle SYSTEM "eagle.dtd">
-<eagle version="6.2">
+<eagle version="6.5.0">
 <drawing>
 <settings>
@@
 <part name="GND30" library="Supply" deviceset="GND" device=""/>
 <part name="ANT4" library="Mechanical" deviceset="ANTENNA" device=""/>
-<part name="R6" library="Passive" deviceset="RES" device="0603" value="50k"/>
-<part name="R25" library="Passive" deviceset="RES" device="0603" value="50k"/>
 <part name="C5" library="Passive" deviceset="CAP" device="0603" value="1uf"/>
 <part name="GND31" library="Supply" deviceset="GND" device=""/>
@@
 <instance part="GND30" gate="1" x="114.3" y="-86.36"/>
 <instance part="ANT4" gate="G$1" x="-200.66" y="-50.8"/>
-<instance part="R6" gate="G$1" x="106.68" y="-71.12" rot="R90"/>
-<instance part="R25" gate="G$1" x="60.96" y="-71.12" rot="R90"/>
 <instance part="C5" gate="G$1" x="223.52" y="-53.34" rot="R270"/>
 <instance part="GND31" gate="1" x="215.9" y="-53.34" rot="R270"/>
@@
 <segment>
 <pinref part="U5" gate="G$1" pin="OUT"/>
-<wire x1="73.66" y1="-78.74" x2="60.96" y2="-78.74" width="0.1524" layer="91"/>
+<wire x1="73.66" y1="-78.74" x2="53.34" y2="-78.74" width="0.1524" layer="91"/>
 <label x="53.34" y="-78.74" size="1.778" layer="91" rot="R180" xref="yes"/>
-<pinref part="R25" gate="G$1" pin="1"/>
-<wire x1="60.96" y1="-78.74" x2="53.34" y2="-78.74" width="0.1524" layer="91"/>
-<wire x1="60.96" y1="-78.74" x2="60.96" y2="-76.2" width="0.1524" layer="91"/>
-<junction x="60.96" y="-78.74"/>
 </segment>
 </net>
@@
 <segment>
 <pinref part="U6" gate="G$1" pin="OUT"/>
-<wire x1="119.38" y1="-78.74" x2="106.68" y2="-78.74" width="0.1524" layer="91"/>
+<wire x1="119.38" y1="-78.74" x2="99.06" y2="-78.74" width="0.1524" layer="91"/>
 <label x="99.06" y="-78.74" size="1.778" layer="91" rot="R180" xref="yes"/>
-<pinref part="R6" gate="G$1" pin="1"/>
-<wire x1="106.68" y1="-78.74" x2="99.06" y2="-78.74" width="0.1524" layer="91"/>
-<wire x1="106.68" y1="-78.74" x2="106.68" y2="-76.2" width="0.1524" layer="91"/>
-<junction x="106.68" y="-78.74"/>
 </segment>
 </net>
@@
 <pinref part="U5" gate="G$1" pin="VCC"/>
 <wire x1="73.66" y1="-73.66" x2="68.58" y2="-73.66" width="0.1524" layer="91"/>
-<wire x1="68.58" y1="-73.66" x2="68.58" y2="-63.5" width="0.1524" layer="91"/>
-<pinref part="R25" gate="G$1" pin="2"/>
-<wire x1="68.58" y1="-63.5" x2="68.58" y2="-60.96" width="0.1524" layer="91"/>
-<wire x1="60.96" y1="-66.04" x2="60.96" y2="-63.5" width="0.1524" layer="91"/>
-<wire x1="60.96" y1="-63.5" x2="68.58" y2="-63.5" width="0.1524" layer="91"/>
-<junction x="68.58" y="-63.5"/>
+<wire x1="68.58" y1="-73.66" x2="68.58" y2="-60.96" width="0.1524" layer="91"/>
 <label x="68.58" y="-60.96" size="1.778" layer="91" rot="R90" xref="yes"/>
 </segment>
@@
 <pinref part="U6" gate="G$1" pin="VCC"/>
 <wire x1="119.38" y1="-73.66" x2="114.3" y2="-73.66" width="0.1524" layer="91"/>
-<wire x1="114.3" y1="-73.66" x2="114.3" y2="-63.5" width="0.1524" layer="91"/>
-<pinref part="R6" gate="G$1" pin="2"/>
-<wire x1="114.3" y1="-63.5" x2="114.3" y2="-60.96" width="0.1524" layer="91"/>
-<wire x1="106.68" y1="-66.04" x2="106.68" y2="-63.5" width="0.1524" layer="91"/>
-<wire x1="106.68" y1="-63.5" x2="114.3" y2="-63.5" width="0.1524" layer="91"/>
-<junction x="114.3" y="-63.5"/>
+<wire x1="114.3" y1="-73.66" x2="114.3" y2="-60.96" width="0.1524" layer="91"/>
 <label x="114.3" y="-60.96" size="1.778" layer="91" rot="R90" xref="yes"/>
 </segment>

Commit message: more
Parts:
- added H3, H4: MOUNTINGHOLE, Mechanical:MOUNTINGHOLE
Changed lines of the file:
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@@
 <part name="P+21" library="Supply" deviceset="+VRAW" device=""/>
 <part name="M1" library="Mechanical" deviceset="VIBMOTOR" device=""/>
+<part name="H3" library="Mechanical" deviceset="MOUNTINGHOLE" device=""/>
+<part name="H4" library="Mechanical" deviceset="MOUNTINGHOLE" device=""/>
 </parts>
 <sheets>
@@
 <instance part="P+21" gate="G$1" x="-149.86" y="-93.98" rot="MR0"/>
 <instance part="M1" gate="G$1" x="-167.64" y="-104.14" rot="MR0"/>
+<instance part="H3" gate="G$1" x="91.44" y="124.46"/>
+<instance part="H4" gate="G$1" x="96.52" y="124.46"/>
 </instances>
 <busses>
