File: Circuits/Boards R3/Swarm Board_3.brd (EAGLE design)
At the start: 56.1 x 63.5 mm, 139 parts, among them CON1 ISP(2X3), CON2 MAIN_CONNECTOR_14SMD, CON4 HEADER_3X1, CON5 HEADER_3X1, CON7 MAIN_CONNECTOR_8, M1 VIBMOTOR, T1 TEFT4300, T10 TEFT4300, T11 NPN2N2222, T12 SI2333DS-T1, T13 NPN2N2222, T14 NPN2N2222, T15 NPN2N2222, T16 NPN2N2222, T17 NPN2N2222, T18 NPN2N2222, T19 IRLML6244TR, T2 TEFT4300, T20 IRLML6244TR, T21 IRLML6244TR, T22 IRLML6244TR, T23 IRLML6244TR, T3 NPN2N2222, T4 TEFT4300, T5 TEFT4300, T6 TEFT4300, T7 TEFT4300, T8 TEFT4300, T9 TEFT4300, U1 ATMEGA324P, U2 MCP73833, U3 ATMEGA1281, U4 MCP9700A, U5 AH182, U6 AH182, U7 QRE1113, U8 QRE1113, U9 QRE1113

Commit message: more
Parts:
- removed R25, R6: 50k, Passive:0603
- moved CON2 1.27 mm to (31.8, 43.2)
Connections:
- net +VSENSE: no longer R25.2, R6.2
- net ENCA: no longer R25.1
- net ENCB: no longer R6.1
Changed lines of the file:
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@@
 <?xml version="1.0" encoding="utf-8"?>
 <!DOCTYPE eagle SYSTEM "eagle.dtd">
-<eagle version="6.2">
+<eagle version="6.5.0">
 <drawing>
 <settings>
@@
 </class>
 </classes>
-<designrules>
+<designrules name="SparkFunDRC">
 <description language="en">&lt;b&gt;EAGLE Design Rules&lt;/b&gt;
 &lt;p&gt;
@@
 <element name="U6" library="Passive" package="3PINHEADER_.100&quot;" value="AH182" x="50.165" y="39.37" rot="R270"/>
 <element name="ANT4" library="Mechanical" package="ANTENNA" value="ANTENNA" x="35.98333125" y="50.8" rot="MR0"/>
-<element name="R6" library="Passive" package="0603" value="50k" x="-28.448" y="-19.685"/>
-<element name="R25" library="Passive" package="0603" value="50k" x="-31.369" y="-19.685"/>
 <element name="C5" library="Passive" package="0603" value="1uf" x="-34.417" y="-36.957"/>
 <element name="C14" library="Passive" package="0603" value="1uf" x="84.582" y="34.925" rot="R180"/>
@@
 <element name="R44" library="Passive" package="0603" value="4.7k" x="16.361853125" y="49.608134375" rot="R225"/>
 <element name="R45" library="Passive" package="0603" value="4.7k" x="47.13176875" y="13.8400375" rot="R45"/>
-<element name="CON2" library="Mechanical" package="FEMALE_HEADER_2MM_2X7_SMD" value="MAIN_CONNECTOR_14SMD" x="31.75" y="44.45" rot="MR0"/>
+<element name="CON2" library="Mechanical" package="FEMALE_HEADER_2MM_2X7_SMD" value="MAIN_CONNECTOR_14SMD" x="31.75" y="43.18" rot="MR0"/>
 <element name="CON7" library="Mechanical" package="FEMALE_HEADER_2MM_2X4" value="MAIN_CONNECTOR_8" x="86.487" y="26.035"/>
 <element name="R46" library="Passive" package="0603" value="100" x="49.682071875" y="16.346121875" rot="R225"/>
@@
 <contactref element="U1" pad="36"/>
 <contactref element="CON2" pad="4"/>
-<wire x1="31.75" y1="42.05" x2="38.113" y2="67.529" width="0" layer="19" extent="1-16"/>
+<wire x1="31.75" y1="40.78" x2="38.113" y2="67.529" width="0" layer="19" extent="1-16"/>
 </signal>
 <signal name="LINESENSE2">
 <contactref element="U1" pad="35"/>
 <contactref element="CON2" pad="3"/>
-<wire x1="33.75" y1="42.05" x2="37.313" y2="67.529" width="0" layer="19" extent="1-16"/>
+<wire x1="33.75" y1="40.78" x2="37.313" y2="67.529" width="0" layer="19" extent="1-16"/>
 </signal>
 <signal name="DATAANTENNA">
@@
 </polygon>
 <contactref element="CON2" pad="13"/>
-<wire x1="59.614" y1="78.744" x2="35.75" y2="46.85" width="0" layer="19" extent="1-16"/>
+<wire x1="59.614" y1="78.744" x2="35.75" y2="45.58" width="0" layer="19" extent="1-16"/>
 </signal>
 <signal name="MA-">
@@
 </polygon>
 <contactref element="CON2" pad="14"/>
-<wire x1="59.614" y1="76.144" x2="37.75" y2="46.85" width="0" layer="19" extent="1-16"/>
+<wire x1="59.614" y1="76.144" x2="37.75" y2="45.58" width="0" layer="19" extent="1-16"/>
 </signal>
 <signal name="MB+">
@@
 </polygon>
 <contactref element="CON2" pad="2"/>
-<wire x1="59.614" y1="72.244" x2="35.75" y2="42.05" width="0" layer="19" extent="1-16"/>
+<wire x1="59.614" y1="72.244" x2="35.75" y2="40.78" width="0" layer="19" extent="1-16"/>
 </signal>
 <signal name="MB-">
@@
 </polygon>
 <contactref element="CON2" pad="1"/>
-<wire x1="59.614" y1="74.844" x2="37.75" y2="42.05" width="0" layer="19" extent="1-16"/>
+<wire x1="59.614" y1="74.844" x2="37.75" y2="40.78" width="0" layer="19" extent="1-16"/>
 </signal>
 <signal name="LED1">
@@
 <contactref element="U1" pad="33"/>
 <contactref element="CON2" pad="5"/>
-<wire x1="29.75" y1="42.05" x2="34.763" y2="69.279" width="0" layer="19" extent="1-16"/>
+<wire x1="29.75" y1="40.78" x2="34.763" y2="69.279" width="0" layer="19" extent="1-16"/>
 </signal>
 <signal name="BIN2">
@@
 <signal name="ENCA">
 <contactref element="U5" pad="3"/>
-<contactref element="R25" pad="1"/>
-<wire x1="6.35" y1="27.2415" x2="-32.119" y2="-19.685" width="0" layer="19" extent="1-1"/>
 </signal>
 <signal name="ENCB">
 <contactref element="U6" pad="3"/>
-<contactref element="R6" pad="1"/>
-<wire x1="-29.198" y1="-19.685" x2="50.165" y2="36.83" width="0" layer="19" extent="1-1"/>
 </signal>
 <signal name="SCL">
@@
 <contactref element="CON4" pad="1"/>
 <contactref element="CON2" pad="7"/>
-<wire x1="25.75" y1="42.05" x2="78.486" y2="41.529" width="0" layer="19" extent="16-16"/>
+<wire x1="25.75" y1="40.78" x2="78.486" y2="41.529" width="0" layer="19" extent="16-16"/>
 </signal>
 <signal name="SGND">
@@
 <contactref element="U4" pad="1"/>
 <contactref element="U5" pad="1"/>
-<contactref element="R25" pad="2"/>
 <contactref element="U6" pad="1"/>
-<contactref element="R6" pad="2"/>
 <contactref element="PR1" pad="2"/>
 <contactref element="C4" pad="1"/>
@@
 <wire x1="26.67" y1="57.15" x2="34.29" y2="57.15" width="0" layer="19" extent="1-1"/>
 <wire x1="15.831521875" y1="49.077803125" x2="26.67" y2="57.15" width="0" layer="19" extent="1-1"/>
-<wire x1="27.75" y1="42.05" x2="15.831521875" y2="49.077803125" width="0" layer="19" extent="1-16"/>
+<wire x1="27.75" y1="40.78" x2="15.831521875" y2="49.077803125" width="0" layer="19" extent="1-16"/>
 <wire x1="50.68156875" y1="14.63316875" x2="51.406421875" y2="30.6585" width="0" layer="19" extent="1-1"/>
 <wire x1="47.662096875" y1="14.370365625" x2="50.68156875" y2="14.63316875" width="0" layer="19" extent="1-1"/>
@@
 <wire x1="30.722" y1="8.255" x2="14.749725" y2="12.93829375" width="0" layer="19" extent="1-1"/>
 <wire x1="-3.241" y1="-17.542" x2="14.749725" y2="12.93829375" width="0" layer="19" extent="1-1"/>
-<wire x1="-27.698" y1="-19.685" x2="-3.241" y2="-17.542" width="0" layer="19" extent="1-1"/>
-<wire x1="-30.619" y1="-19.685" x2="-27.698" y2="-19.685" width="0" layer="19" extent="1-1"/>
-<wire x1="-35.167" y1="-36.957" x2="-30.619" y2="-19.685" width="0" layer="19" extent="1-1"/>
+<wire x1="-35.167" y1="-36.957" x2="-3.241" y2="-17.542" width="0" layer="19" extent="1-1"/>
 <wire x1="-42.279" y1="-36.957" x2="-35.167" y2="-36.957" width="0" layer="19" extent="1-1"/>
 </signal>

Commit message: more stuff dimensions and things
Parts:
- moved H2 14.6 mm to (57.1, 23.5)
- moved U6 7.01 mm to (57.1, 40.0), turned to 90 degrees
- moved ANT2 1.27 mm to (43.2, 50.8)
- moved ANT3 1.27 mm to (20.3, 50.8)
- moved H1 0.64 mm to (6.35, 40.0)
- moved ANT1 0.64 mm to (28.2, 50.8)
- moved ANT4 0.63 mm to (35.3, 50.8)
Changed lines of the file:
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@@
 <attribute name="VALUE" x="72.517" y="26.216" size="0.4064" layer="27" rot="R270"/>
 </element>
-<element name="ANT1" library="Mechanical" package="ANTENNA" value="ANTENNA" x="27.516659375" y="50.8" smashed="yes">
-<attribute name="NAME" x="26.246659375" y="52.07" size="0.6096" layer="25"/>
-<attribute name="VALUE" x="26.246659375" y="48.895" size="0.6096" layer="27"/>
-</element>
-<element name="ANT2" library="Mechanical" package="ANTENNA" value="ANTENNA" x="44.45" y="50.8" smashed="yes">
-<attribute name="NAME" x="43.18" y="52.07" size="0.6096" layer="25"/>
-<attribute name="VALUE" x="43.18" y="48.895" size="0.6096" layer="27"/>
-</element>
-<element name="ANT3" library="Mechanical" package="ANTENNA" value="ANTENNA" x="19.05" y="50.8" smashed="yes">
-<attribute name="NAME" x="17.78" y="52.07" size="0.6096" layer="25"/>
-<attribute name="VALUE" x="17.78" y="48.895" size="0.6096" layer="27"/>
-</element>
-<element name="H1" library="Mechanical" package="MOUNTINGHOLE" value="MOUNTINGHOLE" x="6.35" y="39.37" smashed="yes"/>
-<element name="H2" library="Mechanical" package="MOUNTINGHOLE" value="MOUNTINGHOLE" x="57.15" y="38.1" smashed="yes"/>
+<element name="ANT1" library="Mechanical" package="ANTENNA" value="ANTENNA" x="28.151659375" y="50.8" smashed="yes">
+<attribute name="NAME" x="26.881659375" y="52.07" size="0.6096" layer="25"/>
+<attribute name="VALUE" x="26.881659375" y="48.895" size="0.6096" layer="27"/>
+</element>
+<element name="ANT2" library="Mechanical" package="ANTENNA" value="ANTENNA" x="43.18" y="50.8" smashed="yes">
+<attribute name="NAME" x="41.91" y="52.07" size="0.6096" layer="25"/>
+<attribute name="VALUE" x="41.91" y="48.895" size="0.6096" layer="27"/>
+</element>
+<element name="ANT3" library="Mechanical" package="ANTENNA" value="ANTENNA" x="20.32" y="50.8" smashed="yes">
+<attribute name="NAME" x="19.05" y="52.07" size="0.6096" layer="25"/>
+<attribute name="VALUE" x="19.05" y="48.895" size="0.6096" layer="27"/>
+</element>
+<element name="H1" library="Mechanical" package="MOUNTINGHOLE" value="MOUNTINGHOLE" x="6.35" y="40.005" smashed="yes"/>
+<element name="H2" library="Mechanical" package="MOUNTINGHOLE" value="MOUNTINGHOLE" x="57.15" y="23.495" smashed="yes"/>
 <element name="T13" library="Passive" package="SOT23" value="NPN2N2222" x="40.005" y="57.0865" smashed="yes" rot="R270">
 <attribute name="VALUE" x="37.605" y="58.6865" size="0.6096" layer="27" rot="R270"/>
@@
 <element name="U4" library="Passive" package="SOT23" value="MCP9700A" x="-4.191" y="-18.542"/>
 <element name="U5" library="Passive" package="3PINHEADER_.100&quot;" value="AH182" x="6.35" y="24.7015" rot="R90"/>
-<element name="U6" library="Passive" package="3PINHEADER_.100&quot;" value="AH182" x="50.165" y="39.37" rot="R270"/>
-<element name="ANT4" library="Mechanical" package="ANTENNA" value="ANTENNA" x="35.98333125" y="50.8" rot="MR0"/>
+<element name="U6" library="Passive" package="3PINHEADER_.100&quot;" value="AH182" x="57.15" y="40.005" rot="R90"/>
+<element name="ANT4" library="Mechanical" package="ANTENNA" value="ANTENNA" x="35.34833125" y="50.8" rot="MR0"/>
 <element name="C5" library="Passive" package="0603" value="1uf" x="-34.417" y="-36.957"/>
 <element name="C14" library="Passive" package="0603" value="1uf" x="84.582" y="34.925" rot="R180"/>
@@
 <contactref element="T23" pad="2"/>
 <contactref element="C16" pad="2"/>
+<contactref element="ANT3" pad="P$2"/>
 <wire x1="-59.6385" y1="-100.965" x2="-67.5615" y2="-101.2985" width="0" layer="19" extent="1-1"/>
 <wire x1="-43.827" y1="-36.957" x2="-59.6385" y2="-100.965" width="0" layer="19" extent="1-1"/>
@@
 <wire x1="9.404" y1="-5.204" x2="1.404" y2="-5.204" width="0" layer="19" extent="1-1"/>
 <wire x1="10.6045" y1="13.589" x2="9.404" y2="-5.204" width="0" layer="19" extent="1-1"/>
-<wire x1="15.478359375" y1="52.7361625" x2="19.05" y2="50.8" width="0" layer="19" extent="1-1"/>
+<wire x1="15.478359375" y1="52.7361625" x2="20.32" y2="50.8" width="0" layer="19" extent="1-1"/>
 <wire x1="43.881" y1="6.588" x2="48.142571875" y2="10.702071875" width="0" layer="19" extent="1-1"/>
 <wire x1="37.6715" y1="3.302" x2="43.881" y2="6.588" width="0" layer="19" extent="1-1"/>
-<wire x1="22.6085" y1="58.658" x2="30.734" y2="56.769" width="0" layer="19" extent="1-1"/>
-<wire x1="52.847671875" y1="48.10596875" x2="50.165" y2="39.37" width="0" layer="19" extent="1-1"/>
+<wire x1="22.6085" y1="58.658" x2="20.32" y2="50.8" width="0" layer="19" extent="1-1"/>
+<wire x1="52.847671875" y1="48.10596875" x2="57.15" y2="40.005" width="0" layer="19" extent="1-1"/>
 <wire x1="41.005" y1="58.0365" x2="31.369" y2="57.404" width="0" layer="19" extent="1-1"/>
 <wire x1="42.6085" y1="57.8365" x2="41.005" y2="58.0365" width="0" layer="19" extent="1-1"/>
+<wire x1="66.421" y1="43.999" x2="57.15" y2="40.005" width="0" layer="19" extent="1-1"/>
+<wire x1="67.691" y1="35.064" x2="67.58" y2="42.84" width="0" layer="19" extent="1-1"/>
+<wire x1="76.012" y1="32.124" x2="75.311" y2="35.064" width="0" layer="19" extent="1-1"/>
+<wire x1="73.787" y1="24.396" x2="75.962" y2="30.099" width="0" layer="19" extent="1-1"/>
+<wire x1="67.437" y1="22.987" x2="71.374" y2="23.749" width="0" layer="19" extent="1-1"/>
+<wire x1="69.85" y1="18.161" x2="67.437" y2="22.987" width="0" layer="19" extent="1-1"/>
+<wire x1="63.119" y1="18.808" x2="67.437" y2="22.987" width="0" layer="19" extent="1-1"/>
+<wire x1="63.119" y1="13.855" x2="63.119" y2="18.808" width="0" layer="19" extent="1-1"/>
 <wire x1="7.82408125" y1="34.97464375" x2="6.35" y2="24.7015" width="0" layer="19" extent="1-1"/>
-<wire x1="54.19965" y1="28.481975" x2="50.165" y2="39.37" width="0" layer="19" extent="1-1"/>
-<wire x1="63.119" y1="18.808" x2="55.86086875" y2="28.2786375" width="0" layer="19" extent="1-1"/>
-<wire x1="63.119" y1="13.855" x2="63.119" y2="18.808" width="0" layer="19" extent="1-1"/>
-<wire x1="67.437" y1="22.987" x2="63.119" y2="18.808" width="0" layer="19" extent="1-1"/>
-<wire x1="71.374" y1="23.749" x2="67.437" y2="22.987" width="0" layer="19" extent="1-1"/>
-<wire x1="69.85" y1="18.161" x2="67.437" y2="22.987" width="0" layer="19" extent="1-1"/>
-<wire x1="75.962" y1="30.099" x2="73.787" y2="24.396" width="0" layer="19" extent="1-1"/>
-<wire x1="75.311" y1="35.064" x2="76.012" y2="32.124" width="0" layer="19" extent="1-1"/>
-<wire x1="67.58" y1="42.84" x2="67.691" y2="35.064" width="0" layer="19" extent="1-1"/>
+<wire x1="55.65753125" y1="28.481975" x2="57.15" y2="40.005" width="0" layer="19" extent="1-1"/>
 <wire x1="22.672" y1="74.152" x2="22.745" y2="60.1345" width="0" layer="19" extent="1-1"/>
 <wire x1="59.614" y1="73.544" x2="42.6085" y2="57.8365" width="0" layer="19" extent="1-1"/>
 <wire x1="64.516" y1="80.899" x2="60.859" y2="77.444" width="0" layer="19" extent="1-1"/>
 <wire x1="66.37" y1="75.494" x2="61.087" y2="74.422" width="0" layer="19" extent="1-1"/>
-<contactref element="ANT3" pad="P$2"/>
 </signal>
 <signal name="+VBAT">
@@
 <wire x1="73.152" y1="41.783" x2="73.406" y2="42.037" width="0.4064" layer="1"/>
 <wire x1="73.406" y1="42.037" x2="73.406" y2="42.672" width="0.4064" layer="1"/>
-<wire x1="67.945" y1="44.335" x2="27.516659375" y2="50.8" width="0" layer="19" extent="1-1"/>
 <contactref element="ANT1" pad="P$2"/>
+<wire x1="28.151659375" y1="48.006" x2="28.151659375" y2="50.8" width="0" layer="19" extent="1-1"/>
+<wire x1="67.945" y1="44.335" x2="28.151659375" y2="48.006" width="0" layer="19" extent="1-1"/>
 </signal>
 <signal name="CHGDETECT">
@@
 <contactref element="ANT4" pad="P$1"/>
 <contactref element="U3" pad="P$25"/>
-<wire x1="7.004" y1="-20.704" x2="35.98333125" y2="50.8" width="0" layer="19" extent="1-1"/>
 <contactref element="ANT4" pad="P$2"/>
+<wire x1="35.34833125" y1="48.006" x2="35.34833125" y2="50.8" width="0" layer="19" extent="1-1"/>
+<wire x1="7.004" y1="-20.704" x2="35.34833125" y2="48.006" width="0" layer="19" extent="1-1"/>
 </signal>
 <signal name="SDA">
 <contactref element="ANT2" pad="P$1"/>
 <contactref element="U3" pad="P$26"/>
-<wire x1="7.804" y1="-20.704" x2="44.45" y2="50.8" width="0" layer="19" extent="1-1"/>
 <contactref element="ANT2" pad="P$2"/>
+<wire x1="43.18" y1="48.006" x2="43.18" y2="50.8" width="0" layer="19" extent="1-1"/>
+<wire x1="7.804" y1="-20.704" x2="43.18" y2="48.006" width="0" layer="19" extent="1-1"/>
 </signal>
 <signal name="IRBUMBER">
@@
 <wire x1="12.888628125" y1="48.8258875" x2="13.14054375" y2="49.077803125" width="0.254" layer="1"/>
 <wire x1="13.14054375" y1="49.077803125" x2="15.831521875" y2="49.077803125" width="0.254" layer="1"/>
-<wire x1="49.377184375" y1="50.037065625" x2="69.6595" y2="51.1335" width="0" layer="19" extent="1-1"/>
-<wire x1="50.165" y1="41.91" x2="49.20040625" y2="47.69936875" width="0" layer="19" extent="1-1"/>
-<wire x1="53.178640625" y1="32.934925" x2="50.165" y2="41.91" width="0" layer="19" extent="1-1"/>
+<wire x1="57.15" y1="37.465" x2="69.6595" y2="51.1335" width="0" layer="19" extent="1-1"/>
+<wire x1="53.178640625" y1="32.934925" x2="57.15" y2="37.465" width="0" layer="19" extent="1-1"/>
+<wire x1="49.20040625" y1="47.69936875" x2="57.15" y2="37.465" width="0" layer="19" extent="1-1"/>
 <wire x1="36.588" y1="55.245" x2="48.832709375" y2="50.5815375" width="0" layer="19" extent="1-1"/>
 <wire x1="26.67" y1="57.15" x2="34.29" y2="57.15" width="0" layer="19" extent="1-1"/>

Commit message: more
Parts:
- added H3, H4: MOUNTINGHOLE, Mechanical:MOUNTINGHOLE
Other:
- board size 56.1 x 63.5 mm -> 82.1 x 63.5 mm
Changed lines of the file:
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@@
 <setting verticaltext="up"/>
 </settings>
-<grid distance="0.0025" unitdist="inch" unit="inch" style="lines" multiple="1" display="no" altdistance="0.0005" altunitdist="inch" altunit="inch"/>
+<grid distance="0.1" unitdist="mm" unit="mm" style="lines" multiple="1" display="yes" altdistance="0.0005" altunitdist="inch" altunit="inch"/>
 <layers>
 <layer number="1" name="Top" color="4" fill="1" visible="yes" active="yes"/>
@@
 <wire x1="0" y1="0" x2="63.5" y2="63.5" width="0" layer="47"/>
 <wire x1="0" y1="63.5" x2="63.5" y2="0" width="0" layer="47"/>
+<wire x1="62" y1="18" x2="74.5" y2="18" width="0.2032" layer="20"/>
+<wire x1="74.5" y1="18" x2="74.5" y2="11" width="0.2032" layer="20"/>
+<wire x1="62" y1="18" x2="62" y2="25" width="0.2032" layer="20"/>
+<wire x1="62" y1="25" x2="72" y2="25" width="0.2032" layer="20"/>
+<wire x1="72" y1="25" x2="72" y2="45" width="0.2032" layer="20"/>
+<wire x1="72" y1="45" x2="74.5" y2="45" width="0.2032" layer="20"/>
+<wire x1="74.5" y1="45" x2="74.5" y2="52" width="0.2032" layer="20"/>
+<wire x1="74.5" y1="52" x2="78.331" y2="52" width="0.2032" layer="20"/>
+<wire x1="74.5" y1="11" x2="78.331" y2="11" width="0.2032" layer="20"/>
+<wire x1="78.331" y1="52" x2="78.331" y2="11" width="0.2032" layer="20" curve="-80.43"/>
 </plain>
 <attributes>
@@
 <element name="C16" library="Passive" package="0603" value="1uf" x="-60.3885" y="-100.965"/>
 <element name="M1" library="Mechanical" package="VIBMOTOR" value="VIBMOTOR" x="-72.3265" y="-93.9165"/>
+<element name="H3" library="Mechanical" package="MOUNTINGHOLE" value="MOUNTINGHOLE" x="77" y="15.25"/>
+<element name="H4" library="Mechanical" package="MOUNTINGHOLE" value="MOUNTINGHOLE" x="77" y="48.25"/>
 </elements>
 <signals>

Commit message: fixed derp
Parts:
- moved CON7 24.3 mm to (67.0, 40.6)
Other:
- outline, holes or cut-outs redrawn
Changed lines of the file:
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@@
 <setting verticaltext="up"/>
 </settings>
-<grid distance="0.1" unitdist="mm" unit="mm" style="lines" multiple="1" display="yes" altdistance="0.0005" altunitdist="inch" altunit="inch"/>
+<grid distance="1" unitdist="mm" unit="mm" style="lines" multiple="1" display="yes" altdistance="0.0005" altunitdist="inch" altunit="inch"/>
 <layers>
 <layer number="1" name="Top" color="4" fill="1" visible="yes" active="yes"/>
@@
 <wire x1="0" y1="0" x2="63.5" y2="63.5" width="0" layer="47"/>
 <wire x1="0" y1="63.5" x2="63.5" y2="0" width="0" layer="47"/>
-<wire x1="62" y1="18" x2="74.5" y2="18" width="0.2032" layer="20"/>
 <wire x1="74.5" y1="18" x2="74.5" y2="11" width="0.2032" layer="20"/>
-<wire x1="62" y1="18" x2="62" y2="25" width="0.2032" layer="20"/>
-<wire x1="62" y1="25" x2="72" y2="25" width="0.2032" layer="20"/>
-<wire x1="72" y1="25" x2="72" y2="45" width="0.2032" layer="20"/>
-<wire x1="72" y1="45" x2="74.5" y2="45" width="0.2032" layer="20"/>
+<wire x1="62" y1="36" x2="62" y2="45" width="0.2032" layer="20"/>
+<wire x1="62" y1="45" x2="74.5" y2="45" width="0.2032" layer="20"/>
 <wire x1="74.5" y1="45" x2="74.5" y2="52" width="0.2032" layer="20"/>
 <wire x1="74.5" y1="52" x2="78.331" y2="52" width="0.2032" layer="20"/>
 <wire x1="74.5" y1="11" x2="78.331" y2="11" width="0.2032" layer="20"/>
 <wire x1="78.331" y1="52" x2="78.331" y2="11" width="0.2032" layer="20" curve="-80.43"/>
+<wire x1="62" y1="36" x2="72" y2="36" width="0.2032" layer="20"/>
+<wire x1="72" y1="36" x2="72" y2="18" width="0.2032" layer="20"/>
+<wire x1="72" y1="18" x2="74.5" y2="18" width="0.2032" layer="20"/>
 </plain>
 <attributes>
@@
 <element name="R45" library="Passive" package="0603" value="4.7k" x="47.13176875" y="13.8400375" rot="R45"/>
 <element name="CON2" library="Mechanical" package="FEMALE_HEADER_2MM_2X7_SMD" value="MAIN_CONNECTOR_14SMD" x="31.75" y="43.18" rot="MR0"/>
-<element name="CON7" library="Mechanical" package="FEMALE_HEADER_2MM_2X4" value="MAIN_CONNECTOR_8" x="86.487" y="26.035"/>
+<element name="CON7" library="Mechanical" package="FEMALE_HEADER_2MM_2X4" value="MAIN_CONNECTOR_8" x="66.987" y="40.585"/>
 <element name="R46" library="Passive" package="0603" value="100" x="49.682071875" y="16.346121875" rot="R225"/>
 <element name="R47" library="Passive" package="0603" value="100" x="13.89076875" y="47.159803125" rot="R45"/>
@@
 <contactref element="CON7" pad="8"/>
 <wire x1="83.832" y1="30.48" x2="89.142" y2="30.48" width="0" layer="19" extent="1-1"/>
-<wire x1="83.487" y1="28.435" x2="83.832" y2="30.48" width="0" layer="19" extent="1-1"/>
+<wire x1="63.987" y1="42.985" x2="83.832" y2="30.48" width="0" layer="19" extent="1-1"/>
 <wire x1="83.832" y1="32.639" x2="83.832" y2="30.48" width="0" layer="19" extent="1-1"/>
 <wire x1="83.832" y1="34.925" x2="83.832" y2="32.639" width="0" layer="19" extent="1-1"/>
@@
 <contactref element="R2" pad="1"/>
 <contactref element="CON7" pad="2"/>
-<wire x1="85.487" y1="23.635" x2="89.142" y2="32.639" width="0" layer="19" extent="1-1"/>
+<wire x1="65.987" y1="38.185" x2="89.142" y2="32.639" width="0" layer="19" extent="1-1"/>
 </signal>
 <signal name="S+VSENSE">
@@
 <wire x1="91.726" y1="23.103" x2="95.726" y2="24.903" width="0" layer="19" extent="1-1"/>
 <wire x1="84.951" y1="18.542" x2="91.726" y2="23.103" width="0" layer="19" extent="1-1"/>
-<wire x1="83.487" y1="23.635" x2="84.951" y2="18.542" width="0" layer="19" extent="1-1"/>
+<wire x1="63.987" y1="38.185" x2="84.951" y2="18.542" width="0" layer="19" extent="1-1"/>
 </signal>
 <signal name="LEFTBUMPER">
@@
 <contactref element="CON7" pad="3"/>
 <contactref element="U8" pad="P$4"/>
-<wire x1="87.487" y1="23.635" x2="85.332" y2="32.639" width="0" layer="19" extent="1-1"/>
-<wire x1="91.726" y1="24.903" x2="87.487" y2="23.635" width="0" layer="19" extent="1-1"/>
+<wire x1="67.987" y1="38.185" x2="85.332" y2="32.639" width="0" layer="19" extent="1-1"/>
+<wire x1="91.726" y1="24.903" x2="67.987" y2="38.185" width="0" layer="19" extent="1-1"/>
 </signal>
 <signal name="SLEFTBUMPER">
@@
 <contactref element="U9" pad="P$4"/>
 <contactref element="R34" pad="2"/>
-<wire x1="89.487" y1="28.435" x2="91.853" y2="34.809" width="0" layer="19" extent="1-1"/>
-<wire x1="85.332" y1="30.48" x2="89.487" y2="28.435" width="0" layer="19" extent="1-1"/>
+<wire x1="69.987" y1="42.985" x2="91.853" y2="34.809" width="0" layer="19" extent="1-1"/>
+<wire x1="85.332" y1="30.48" x2="69.987" y2="42.985" width="0" layer="19" extent="1-1"/>
 </signal>
 <signal name="MOSI">
